File: Test/Test_Measurement/Current_Measurement.kicad_sch (KiCad schematic)
At the start: 15 parts, among them U2 OP07CP

Commit message: Update PCB
Parts:
- R6, R7: value 680K/1%/1_8W -> 620K/1%/1_8W
Connections:
- net N_Rshunt: now also R3.2; no longer R3.1
- net at F1.2, R2.2, R4.1: now also R3.1; no longer R3.2
- no-connect marks 0 -> 2
Other:
- note added: "Hồi tiếp âm"
