File: Test/Test_Measurement/Test_Measurement.kicad_pcb (KiCad board)
At the start: 2 copper layers, 100 x 100 mm, 94 parts, among them J1 Barrel_Jack_Switch, J2 Conn_01x02_Socket, J3 Conn_01x03_Socket, J4 Conn_01x02_Socket, K1 EA2-5NJ, Q1 MMBT2222A, Q2 MMBT2222A, Q3 MMBT2222A, SW1 SW_Push, U1 STM32F103C8T6_Bluepill, U10 ICL7662CBA, U11 PC817X2NIPW, U2 OP07CP, U3 OP07CP, U4 LM358N/P, U5 LM358N/P, U6 LM358N/P, U7 LM1117IMP-5.0, U8 LD1117S33CTR_SOT223, U9 L7809CV

Commit message: Update PCB
Parts:
- removed C1, C31, C32, C39, C40: 10uF/16V, Measure_Power_AC:Ceramic_Cap_0805
- removed C2, C34, C35, C36, C37: 100nF/50V, Measure_Power_AC:Ceramic_Cap_0805
- removed U7: LM1117IMP-5.0, Measure_Power_AC:SOT-223
- removed U8: LD1117S33CTR_SOT223, Measure_Power_AC:SOT-223
- added D8: LED_5, Measure_Power_AC:LED_D5.0mm, F.Cu at (122.7, 34.3)
- added R24: 1K/1%/1_8W, Measure_Power_AC:Res_0805, B.Cu at (117.2, 35.7)
- C10, C11, C12, C13, C14, C15, C16, C17, C18, C19, C20, C21, C22, C23, C24, C25, C26, C27, C28, C29, C3, C30, C33, C38, C4, C41, C5, C6, C7, C8, C9, D1, D2, D3, D4, D5, D6, D7, Q1, Q2, Q3, R1, R10, R11, R12, R13, R14, R15, R16, R17, R18, R19, R20, R21, R22, R23, R4, R5, R8, R9, U10, U11: moved to B.Cu
- C42, C43: footprint Capacitor_SMD:CP_Elec_4x5.4 -> Measure_Power_AC:Tan_Cap_A; moved to B.Cu
- J1: footprint Connector_BarrelJack:BarrelJack_GCT_DCJ200-10-A_Horizontal -> Measure_Power_AC:XKB_DC-005-5A-2.0
- J2, J4: footprint Connector_Phoenix_MC:PhoenixContact_MC_1,5_2-G-3.81_1x02_P3.81mm_Horizontal -> Connector_Phoenix_MC_HighVoltage:PhoenixContact_MC_1,5_2-G-5.08_1x02_P5.08mm_Horizontal
- R6, R7: value 680K/1%/1_8W -> 620K/1%/1_8W; moved to B.Cu
- SW1: value SW_Push -> Button_6mm; footprint Measure_Power_AC:SW_SMD -> Measure_Power_AC:SW_B3F-1060_OMR
- moved C3 231.4 mm to (120.4, 131.2)
- moved R1 230.2 mm to (122.2, 129.9), turned to 180 degrees
- moved SW1 222.7 mm to (116.7, 133.9)
- moved J3 212.1 mm to (122.2, 115.1), turned to -90 degrees
- moved R9 199.3 mm to (77.9, 60.6)
- moved R8 194.0 mm to (73.5, 60.5)
- moved R6 192.2 mm to (77.9, 62.6)
- moved F1 191.7 mm to (73.8, 30.1), turned to 180 degrees
- moved R7 190.6 mm to (73.5, 62.7)
- moved U9 181.4 mm to (113.3, 44.7), turned to -90 degrees
- moved K1 178.3 mm to (65.3, 58.0), turned to 90 degrees
- moved J1 178.2 mm to (113.3, 28.9), turned to -90 degrees
- moved U1 176.1 mm to (87.9, 124.7), turned to 180 degrees
- moved C6 174.7 mm to (86.5, 70.3), turned to 90 degrees
- moved C33 174.2 mm to (112.3, 40.6)
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Connections:
- D7 pad 2: +5V -> +12V
- J1 pad 3: unconnected-(J1-Pad3) -> Relay_1_P
- J3 pad 1: UART1_RX -> Relay_1_P
- J3 pad 2: UART1_TX -> UART3_RX
- J3 pad 3: Relay_1_P -> UART3_TX
- K1 pad 10: +5V -> +12V
- R20 pad 2: +3V3 -> +3.3V
- R21 pad 2: +3V3 -> +3.3V
- R3 pad 1: N_Rshunt -> Net-(F1-Pad2)
- R3 pad 2: Net-(F1-Pad2) -> N_Rshunt
- SW1 pad 1: Relay_1_P -> unconnected-(SW1-Pad1)
- U1 pad 15: unconnected-(U1A-PB10-Pad15) -> UART3_TX
- U1 pad 16: unconnected-(U1A-PB11-Pad16) -> UART3_RX
- U1 pad 18: unconnected-(U1B-3V3-Pad18) -> +3.3V
- U1 pad 26: UART1_TX -> unconnected-(U1A-PA9-Pad26)
- U1 pad 27: UART1_RX -> unconnected-(U1A-PA10-Pad27)
- U1 pad 38: +5V -> unconnected-(U1B-5V-Pad38)
- U1 pad 6: Peak_Voltage -> Peak_Current
- U1 pad 7: Peak_Current -> Peak_Voltage
- U11 pad 4: +5V -> +12V
Routing:
- net Relay_1_P: track 0.00 -> 574.1 mm, vias 0 -> 20
- net N_Rshunt: track 0.00 -> 204.7 mm, vias 0 -> 3
- net +9V: track 0.00 -> 201.4 mm, vias 0 -> 7
- net -9V: track 0.00 -> 158.9 mm, vias 0 -> 7
- net +3.3V: track 0.00 -> 135.2 mm, vias 0 -> 3
- net Net-(F1-Pad2): track 0.00 -> 122.2 mm, vias 0 -> 1
- net +12V: track 0.00 -> 97.1 mm, vias 0 -> 3
- net Current_Sensor: track 0.00 -> 95.0 mm
- net RESET: track 0.00 -> 66.9 mm
- net Relay_Control: track 0.00 -> 62.8 mm
- net UART3_RX: track 0.00 -> 57.9 mm
- net P_Voltage: track 0.00 -> 57.3 mm
- net Voltage_Sensor: track 0.00 -> 56.4 mm, vias 0 -> 2
- net UART3_TX: track 0.00 -> 49.3 mm
- net Peak_Current: track 0.00 -> 38.8 mm
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- added copper zone on B.Cu, net -9V
- added copper zone on B.Cu, net N_Rshunt
- added copper zone on B.Cu, net Net-(F1-Pad2)
- added copper zone on B.Cu, net P_Rshunt
- added copper zone on B.Cu, net P_Voltage
- added copper zone on B.Cu, net Relay_1_P
Other:
- board size 100 x 100 mm -> 106.7 x 117.5 mm
