File: Test/Test_Measurement/Voltage_Measurement.kicad_sch (KiCad schematic)
At the start: 10 parts, among them U3 OP07CP

Commit message: Update PCB
Connections:
- no-connect marks 0 -> 2
Other:
- note added: "Hồi tiếp âm"
Changed lines of the file:
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@@
 		(color 0 0 0 0)
 	)
+	(no_connect
+		(at 129.54 82.55)
+	)
+	(no_connect
+		(at 127 82.55)
+	)
 	(wire
 		(pts
@@
 		)
 	)
+	(text "Hồi tiếp âm"
+		(exclude_from_sim no)
+		(at 158.242 53.34 0)
+		(effects
+			(font
+				(size 1.27 1.27)
+			)
+		)
+	)
