File: Hardware/MEASURE_POWER_AC/Connectors.kicad_sch (KiCad schematic)
At the start: 15 parts, among them J2 Conn_01x02_Pin, J3 Conn_01x03_Pin, J4 Conn_01x02_Pin

Commit message: Update BOM
Changed lines of the file:
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@@
 	(text "~AC~"
 		(exclude_from_sim no)
-		(at 82.804 78.74 0)
+		(at 79.248 78.74 0)
 		(effects
 			(font
