File: Hardware/MEASURE_POWER_AC/ESP32.kicad_sch (KiCad schematic)
At the start: 22 parts, among them SW2 SW_Push, SW3 SW_Push, SW4 Button_12mm, SW5 Button_12mm, U2 ESP32-WROOM-32E__4MB_HIGH_TEM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

Commit message: Update PCB
Parts:
- SW2: value SW_Push -> FLASH
- SW3: value SW_Push -> EN
- SW4: value Button_12mm -> USER_1
- SW5: value Button_12mm -> USER_2
Changed lines of the file:
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@@
 			)
 		)
-		(property "Value" "SW_Push"
+		(property "Value" "FLASH"
 			(at 40.64 46.9899 90)
 			(effects
@@
 			)
 		)
-		(property "Value" "Button_12mm"
+		(property "Value" "USER_2"
 			(at 265.43 55.8799 90)
 			(effects
@@
 			)
 		)
-		(property "Value" "Button_12mm"
+		(property "Value" "USER_1"
 			(at 229.87 55.8799 90)
 			(effects
@@
 			)
 		)
-		(property "Value" "SW_Push"
+		(property "Value" "EN"
 			(at 40.64 100.3299 90)
 			(effects

Commit message: Update BOM
Parts:
- SW2, SW3: Supply URL (none) -> https://www.thegioiic.com/nut-nhan-3x4mm-cao-2-5mm-2-chan-s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; Suppy URL https://www.thegioiic.com/nut-nhan-3x4mm-cao-2-5mm-2-chan-s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 -> (none)
Changed lines of the file:
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@@
 			)
 		)
-		(property "Suppy URL" "https://www.thegioiic.com/nut-nhan-3x4mm-cao-2-5mm-2-chan-smd"
+		(property "Suppy URL" ""
 			(at 33.02 46.736 0)
+			(effects
+				(font
+					(size 1.27 1.27)
+				)
+				(hide yes)
+			)
+		)
+		(property "Supply URL" "https://www.thegioiic.com/nut-nhan-3x4mm-cao-2-5mm-2-chan-smd"
+			(at 39.37 45.72 0)
 			(effects
 				(font
@@
 			)
 		)
-		(property "Suppy URL" "https://www.thegioiic.com/nut-nhan-3x4mm-cao-2-5mm-2-chan-smd"
+		(property "Suppy URL" ""
 			(at 33.02 100.076 0)
 			(effects
 				(font
+					(size 1.27 1.27)
+				)
+				(hide yes)
+			)
+		)
+		(property "Supply URL" "https://www.thegioiic.com/nut-nhan-3x4mm-cao-2-5mm-2-chan-smd"
+			(at 39.37 99.06 0)
+			(effects
+				(font
