File: Hardware/MEASURE_POWER_AC/Peak_Detector.kicad_sch (KiCad schematic)
At the start: 34 parts, among them U10 OP07CSZ, U7 OP07CSZ, U8 OP07CSZ, U9 OP07CSZ

Commit message: Update BOM
Parts:
- U10, U7, U8, U9: Supply name (none) -> tme; Supply name  tme -> (none)
Changed lines of the file:
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@@
 			)
 		)
-		(property "Supply name " "tme"
+		(property "Supply name " ""
 			(at 160.528 154.94 0)
 			(effects
@@
 			)
 		)
+		(property "Supply name" "tme"
+			(at 149.86 146.05 0)
+			(effects
+				(font
+					(size 1.27 1.27)
+				)
+				(hide yes)
+			)
+		)
 		(pin "2"
 		)
@@
 			)
 		)
-		(property "Supply name " "tme"
+		(property "Supply name " ""
 			(at 112.268 86.36 0)
 			(effects
@@
 			)
 		)
+		(property "Supply name" "tme"
+			(at 101.6 77.47 0)
+			(effects
+				(font
+					(size 1.27 1.27)
+				)
+				(hide yes)
+			)
+		)
 		(pin "2"
 		)
@@
 			)
 		)
-		(property "Supply name " "tme"
+		(property "Supply name " ""
 			(at 163.068 83.82 0)
 			(effects
@@
 			)
 		)
+		(property "Supply name" "tme"
+			(at 152.4 74.93 0)
+			(effects
+				(font
+					(size 1.27 1.27)
+				)
+				(hide yes)
+			)
+		)
 		(pin "2"
 		)
@@
 			)
 		)
-		(property "Supply name " "tme"
+		(property "Supply name " ""
 			(at 109.728 157.48 0)
 			(effects
@@
 			(effects
 				(font
+					(size 1.27 1.27)
+				)
+				(hide yes)
+			)
+		)
+		(property "Supply name" "tme"
+			(at 99.06 148.59 0)
+			(effects
+				(font
