File: Hardware/MEASURE_POWER_AC/Voltage_Measurement.kicad_sch (KiCad schematic)
At the start: 18 parts, among them U6 OP07CSZ

Commit message: Update BOM
Parts:
- U6: Supply name (none) -> tme; Supply name  tme -> (none)
Changed lines of the file:
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@@
 			)
 		)
-		(property "Supply name " "tme"
+		(property "Supply name " ""
 			(at 166.878 105.41 0)
 			(effects
@@
 			(effects
 				(font
+					(size 1.27 1.27)
+				)
+				(hide yes)
+			)
+		)
+		(property "Supply name" "tme"
+			(at 156.21 96.52 0)
+			(effects
+				(font
