File: Hardware/MEASURE_POWER_AC/MCU.kicad_sch (KiCad schematic)
At the start: 31 parts, among them J1 Conn_01x04_Pin, SW1 SW_Push, U1 STM32F103C8T6, Y1 Crystal_8MHz_SMD-4PIN

Commit message: Update PCB
Parts:
- removed NT1: NetTie_2, NetTie:NetTie-2_SMD_Pad0.5mm, symbol Device:NetTie_2
- SW1: value SW_Push -> RESET
Connections:
- net GNDA is gone; now on net GND: C15.1, U1.8 (VSSA)
Changed lines of the file:
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@@
 	)
 	(junction
+		(at 143.51 151.13)
+		(diameter 0)
+		(color 0 0 0 0)
+	)
+	(junction
 		(at 101.6 139.7)
 		(diameter 0)
@@
 	)
 	(junction
-		(at 143.51 151.13)
-		(diameter 0)
-		(color 0 0 0 0)
-	)
-	(junction
 		(at 118.11 151.13)
 		(diameter 0)
@@
 	(wire
 		(pts
-			(xy 143.51 151.13) (xy 143.51 152.4)
+			(xy 143.51 148.59) (xy 143.51 151.13)
 		)
 		(stroke
@@
 	(wire
 		(pts
-			(xy 134.62 151.13) (xy 143.51 151.13)
+			(xy 26.67 148.59) (xy 26.67 151.13)
 		)
 		(stroke
@@
 	(wire
 		(pts
-			(xy 26.67 148.59) (xy 26.67 151.13)
+			(xy 81.28 78.74) (xy 92.71 78.74)
 		)
 		(stroke
@@
 	(wire
 		(pts
-			(xy 81.28 78.74) (xy 92.71 78.74)
+			(xy 193.04 39.37) (xy 193.04 43.18)
 		)
 		(stroke
@@
 	(wire
 		(pts
-			(xy 193.04 39.37) (xy 193.04 43.18)
+			(xy 101.6 140.97) (xy 101.6 139.7)
 		)
 		(stroke
@@
 	(wire
 		(pts
-			(xy 101.6 140.97) (xy 101.6 139.7)
+			(xy 143.51 151.13) (xy 143.51 152.4)
 		)
 		(stroke
@@
 	(wire
 		(pts
-			(xy 143.51 151.13) (xy 143.51 148.59)
-		)
-		(stroke
-			(width 0)
-			(type default)
-		)
-	)
-	(wire
-		(pts
 			(xy 138.43 86.36) (xy 160.02 86.36)
 		)
@@
 	(wire
 		(pts
-			(xy 118.11 151.13) (xy 129.54 151.13)
+			(xy 118.11 151.13) (xy 143.51 151.13)
 		)
 		(stroke
@@
 	)
 	(symbol
-		(lib_id "power:GNDA")
-		(at 143.51 152.4 0)
-		(unit 1)
-		(exclude_from_sim no)
-		(in_bom yes)
-		(on_board yes)
-		(dnp no)
-		(fields_autoplaced yes)
-		(property "Reference" "#PWR010"
-			(at 143.51 158.75 0)
-			(effects
-				(font
-					(size 1.27 1.27)
-				)
-				(hide yes)
-			)
-		)
-		(property "Value" "GNDA"
-			(at 143.51 157.48 0)
-			(effects
-				(font
-					(size 1.27 1.27)
-				)
-			)
-		)
-		(property "Footprint" ""
-			(at 143.51 152.4 0)
-			(effects
-				(font
-					(size 1.27 1.27)
-				)
-				(hide yes)
-			)
-		)
-		(property "Datasheet" ""
-			(at 143.51 152.4 0)
-			(effects
-				(font
-					(size 1.27 1.27)
-				)
-				(hide yes)
-			)
-		)
-		(property "Description" "Power symbol creates a global label with name \"GNDA\" , analog ground"
-			(at 143.51 152.4 0)
-			(effects
-				(font
-					(size 1.27 1.27)
-				)
-				(hide yes)
-			)
-		)
-		(pin "1"
-		)
-		(instances
-			(project "MEASURE_POWER_AC"
-				(path "/a4d4b55a-fae9-4c17-8d9b-0fae9d35e0cc/05d0bcbd-9292-4250-a3df-595675932f2e"
-					(reference "#PWR010")
-					(unit 1)
-				)
-			)
-		)
-	)
-	(symbol
 		(lib_id "power:GND")
 		(at 199.39 43.18 0)
@@
 	)
 	(symbol
-		(lib_id "Device:NetTie_2")
-		(at 132.08 151.13 0)
-		(unit 1)
-		(exclude_from_sim no)
-		(in_bom no)
-		(on_board yes)
-		(dnp no)
-		(property "Reference" "NT1"
-			(at 132.08 156.21 0)
-			(effects
-				(font
-					(size 1.27 1.27)
-				)
-			)
-		)
-		(property "Value" "NetTie_2"
-			(at 132.08 153.67 0)
-			(effects
-				(font
-					(size 1.27 1.27)
-				)
-			)
-		)
-		(property "Footprint" "NetTie:NetTie-2_SMD_Pad0.5mm"
-			(at 132.08 151.13 0)
-			(effects
-				(font
-					(size 1.27 1.27)
-				)
-				(hide yes)
-			)
-		)
-		(property "Datasheet" "~"
-			(at 132.08 151.13 0)
-			(effects
-				(font
-					(size 1.27 1.27)
-				)
-				(hide yes)
-			)
-		)
-		(property "Description" "Net tie, 2 pins"
-			(at 132.08 151.13 0)
-			(effects
-				(font
-					(size 1.27 1.27)
-				)
-				(hide yes)
-			)
-		)
-		(pin "2"
-		)
-		(pin "1"
-		)
-		(instances
-			(project ""
-				(path "/a4d4b55a-fae9-4c17-8d9b-0fae9d35e0cc/05d0bcbd-9292-4250-a3df-595675932f2e"
-					(reference "NT1")
-					(unit 1)
-				)
-			)
-		)
-	)
-	(symbol
 		(lib_id "Measurement_Power_AC:Ceramic_Cap_SMD_1uF_16V")
 		(at 40.64 30.48 90)
@@
 	)
 	(symbol
-		(lib_id "power:GNDA")
-		(at 193.04 43.18 0)
-		(unit 1)
-		(exclude_from_sim no)
-		(in_bom yes)
-		(on_board yes)
-		(dnp no)
-		(fields_autoplaced yes)
-		(property "Reference" "#PWR014"
-			(at 193.04 49.53 0)
-			(effects
-				(font
-					(size 1.27 1.27)
-				)
-				(hide yes)
-			)
-		)
-		(property "Value" "GNDA"
-			(at 193.04 48.26 0)
-			(effects
-				(font
-					(size 1.27 1.27)
-				)
-			)
-		)
-		(property "Footprint" ""
-			(at 193.04 43.18 0)
-			(effects
-				(font
-					(size 1.27 1.27)
-				)
-				(hide yes)
-			)
-		)
-		(property "Datasheet" ""
-			(at 193.04 43.18 0)
-			(effects
-				(font
-					(size 1.27 1.27)
-				)
-				(hide yes)
-			)
-		)
-		(property "Description" "Power symbol creates a global label with name \"GNDA\" , analog ground"
-			(at 193.04 43.18 0)
-			(effects
-				(font
-					(size 1.27 1.27)
-				)
-				(hide yes)
-			)
-		)
-		(pin "1"
-		)
-		(instances
-			(project ""
-				(path "/a4d4b55a-fae9-4c17-8d9b-0fae9d35e0cc/05d0bcbd-9292-4250-a3df-595675932f2e"
-					(reference "#PWR014")
-					(unit 1)
-				)
-			)
-		)
-	)
-	(symbol
 		(lib_id "Measurement_Power_AC:Res_10K_0603_1%")
 		(at 251.46 96.52 90)
@@
 	(symbol
 		(lib_id "power:GND")
+		(at 193.04 43.18 0)
+		(unit 1)
+		(exclude_from_sim no)
+		(in_bom yes)
+		(on_board yes)
+		(dnp no)
+		(fields_autoplaced yes)
+		(property "Reference" "#PWR014"
+			(at 193.04 49.53 0)
+			(effects
+				(font
+					(size 1.27 1.27)
+				)
+				(hide yes)
+			)
+		)
+		(property "Value" "GND"
+			(at 193.04 48.26 0)
+			(effects
+				(font
+					(size 1.27 1.27)
+				)
+			)
+		)
+		(property "Footprint" ""
+			(at 193.04 43.18 0)
+			(effects
+				(font
+					(size 1.27 1.27)
+				)
+				(hide yes)
+			)
+		)
+		(property "Datasheet" ""
+			(at 193.04 43.18 0)
+			(effects
+				(font
+					(size 1.27 1.27)
+				)
+				(hide yes)
+			)
+		)
+		(property "Description" "Power symbol creates a global label with name \"GND\" , ground"
+			(at 193.04 43.18 0)
+			(effects
+				(font
+					(size 1.27 1.27)
+				)
+				(hide yes)
+			)
+		)
+		(pin "1"
+		)
+		(instances
+			(project "MEASURE_POWER_AC"
+				(path "/a4d4b55a-fae9-4c17-8d9b-0fae9d35e0cc/05d0bcbd-9292-4250-a3df-595675932f2e"
+					(reference "#PWR014")
+					(unit 1)
+				)
+			)
+		)
+	)
+	(symbol
+		(lib_id "power:GND")
 		(at 251.46 114.3 0)
 		(unit 1)
@@
 			)
 		)
-		(property "Value" "SW_Push"
+		(property "Value" "RESET"
 			(at 252.73 106.6799 90)
 			(effects
@@
 					(unit 1)
 				)
+			)
+		)
+	)
+	(symbol
+		(lib_id "power:GND")
+		(at 143.51 152.4 0)
+		(unit 1)
+		(exclude_from_sim no)
+		(in_bom yes)
+		(on_board yes)
+		(dnp no)
+		(fields_autoplaced yes)
+		(property "Reference" "#PWR010"
+			(at 143.51 158.75 0)
+			(effects
+				(font
+					(size 1.27 1.27)
+				)
+				(hide yes)
+			)
+		)
+		(property "Value" "GND"
+			(at 143.51 157.48 0)
+			(effects
+				(font
+					(size 1.27 1.27)
+				)
+			)
+		)
+		(property "Footprint" ""
+			(at 143.51 152.4 0)
+			(effects
+				(font
+					(size 1.27 1.27)
+				)
+				(hide yes)
+			)
+		)
+		(property "Datasheet" ""
+			(at 143.51 152.4 0)
+			(effects
+				(font
+					(size 1.27 1.27)
+				)
+				(hide yes)
+			)
+		)
+		(property "Description" "Power symbol creates a global label with name \"GND\" , ground"
+			(at 143.51 152.4 0)
+			(effects
+				(font
+					(size 1.27 1.27)
+				)
+				(hide yes)
+			)
+		)
+		(pin "1"
+		)
+		(instances
+			(project "MEASURE_POWER_AC"
+				(path "/a4d4b55a-fae9-4c17-8d9b-0fae9d35e0cc/05d0bcbd-9292-4250-a3df-595675932f2e"
+					(reference "#PWR010")
+					(unit 1)
+				)

Commit message: Update BOM
Parts:
- SW1: Supply URL (none) -> https://www.thegioiic.com/nut-nhan-3x4mm-cao-2-5mm-2-chan-s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; Suppy URL https://www.thegioiic.com/nut-nhan-3x4mm-cao-2-5mm-2-chan-s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 -> (none)
- U1: Supply name (none) -> Thegioiic; Supply name  Thegioiic -> (none)
Changed lines of the file:
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@@
 			)
 		)
-		(property "Suppy URL" "https://www.thegioiic.com/nut-nhan-3x4mm-cao-2-5mm-2-chan-smd"
+		(property "Suppy URL" ""
 			(at 245.11 106.426 0)
+			(effects
+				(font
+					(size 1.27 1.27)
+				)
+				(hide yes)
+			)
+		)
+		(property "Supply URL" "https://www.thegioiic.com/nut-nhan-3x4mm-cao-2-5mm-2-chan-smd"
+			(at 251.46 105.41 0)
 			(effects
 				(font
@@
 			)
 		)
-		(property "Supply name " "Thegioiic"
+		(property "Supply name " ""
 			(at 96.52 110.49 0)
 			(effects
@@
 		)
 		(property "Supply URL" "https://www.thegioiic.com/stm32f103c8t6-32-bit-arm-cortex-m3-microcontroller-72mhz-64kb-flash-48-lqfp"
+			(at 96.52 110.49 0)
+			(effects
+				(font
+					(size 1.27 1.27)
+				)
+				(hide yes)
+			)
+		)
+		(property "Supply name" "Thegioiic"
 			(at 96.52 110.49 0)
 			(effects
@@
 			)
 		)
-		(property "Supply name " "Thegioiic"
+		(property "Supply name " ""
 			(at 186.69 45.72 0)
 			(effects
@@
 			(at 186.69 45.72 0)
 			(effects
+				(font
+					(size 1.27 1.27)
+				)
+				(hide yes)
+			)
+		)
+		(property "Supply name" "Thegioiic"
+			(at 186.69 45.72 0)
+			(effects

Commit message: Update
Connections:
- net Zero_Current: now also U1.41 (PB5); no longer U1.42 (PB6)
- net Zero_Voltage: now also U1.42 (PB6); no longer U1.41 (PB5)
Changed lines of the file:
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@@
 		)
 	)
-	(global_label "Zero_Voltage"
+	(global_label "Zero_Current"
 		(shape input)
 		(at 81.28 81.28 180)
@@
 		)
 		(property "Intersheetrefs" "${INTERSHEET_REFS}"
-			(at 66.0788 81.28 0)
+			(at 66.1392 81.28 0)
 			(effects
 				(font
@@
 		)
 	)
-	(global_label "Zero_Current"
+	(global_label "Zero_Voltage"
 		(shape input)
 		(at 81.28 83.82 180)
@@
 		)
 		(property "Intersheetrefs" "${INTERSHEET_REFS}"
-			(at 66.1392 83.82 0)
+			(at 66.0788 83.82 0)
 			(effects
 				(font
