File: Hardware/MEASURE_POWER_AC/Power_Supply.kicad_sch (KiCad schematic)
At the start: 41 parts, among them U12 L78L09_SOT89, U13 TPS54231DR, U14 LM1086RS, U15 L78L05_SOT89, U16 ICL7660CBAZ

Commit message: Update PCB
Parts:
- added D21: 12V, Measure_Power_AC:LED_0805, symbol Measurement_Power_AC:LED_0805
- added D22: 9V, Measure_Power_AC:LED_0805, symbol Measurement_Power_AC:LED_0805
- added D23, D24: 5V, Measure_Power_AC:LED_0805, symbol Measurement_Power_AC:LED_0805
- added D25: -9V, Measure_Power_AC:LED_0805, symbol Measurement_Power_AC:LED_0805
- added D26: 3V3, Measure_Power_AC:LED_0805, symbol Measurement_Power_AC:LED_0805
- added R63, R64, R65, R66, R67, R68: 1K/1%/1_10W, Measure_Power_AC:Res_0603, symbol Measurement_Power_AC:Res_1K_0603_1%
Connections:
- net +12V: now also D21.2 (A)
- net +3V3: now also D26.2 (A)
- net +5V_1: now also D23.2 (A)
- net +5V_2: now also D24.2 (A)
- net +9V: now also D22.2 (A)
- net -9V: now also D25.1 (K)
- net GND: now also R63.2, R64.2, R65.2, R66.2, R67.2, R68.2
- new net: D23.1 (K), R65.1
- new net: D21.1 (K), R63.1
- new net: D26.1 (K), R68.1
- new net: D24.1 (K), R66.1
- new net: D22.1 (K), R64.1
- new net: D25.2 (A), R67.1
Other:
- moved on the sheet: C70, C71, C72, C73, C74, C75, C76, C77, C78, C79, C80, C81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

Commit message: Update
Parts:
- removed U16: ICL7660CBAZ, Measure_Power_AC:SOIC-8, symbol Measurement_Power_AC:ICL7660CBAZ
- added U16: ICL7662CBA-T, Measure_Power_AC:SOIC-8, symbol Measurement_Power_AC:ICL7662CBA-T
Connections:
- net +9V: now also U16.8 (V+)
- net -9V: now also U16.5 (VOUT)
- net GND: now also U16.3 (GND), U16.6 (LV)
- net at C91.1: now also U16.2 (CAP+)
- net at C91.2: now also U16.4 (CAP-)
Other:
- note added: "Charge Pump -9V - ICL7662CBAZ"
- note removed: "Charge Pump -9V - ICL7660CBAZ"
Changed lines of the file:
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@@
 	)
 	(no_connect
-		(at 284.48 83.82)
-	)
-	(no_connect
 		(at 284.48 76.2)
 	)
-	(wire
-		(pts
-			(xy 139.7 90.17) (xy 139.7 92.71)
-		)
-		(stroke
-			(width 0)
-			(type default)
-		)
+	(no_connect
+		(at 284.48 86.36)
 	)
 	(wire
@@
 	(wire
 		(pts
-			(xy 283.21 95.25) (xy 294.64 95.25)
+			(xy 281.94 95.25) (xy 294.64 95.25)
 		)
 		(stroke
@@
 	(wire
 		(pts
+			(xy 281.94 83.82) (xy 284.48 83.82)
+		)
+		(stroke
+			(width 0)
+			(type default)
+		)
+	)
+	(wire
+		(pts
 			(xy 54.61 121.92) (xy 54.61 124.46)
 		)
@@
 	(wire
 		(pts
-			(xy 139.7 92.71) (xy 148.59 92.71)
-		)
-		(stroke
-			(width 0)
-			(type default)
-		)
-	)
-	(wire
-		(pts
 			(xy 379.73 87.63) (xy 387.35 87.63)
 		)
@@
 	(wire
 		(pts
-			(xy 283.21 86.36) (xy 283.21 95.25)
+			(xy 281.94 83.82) (xy 281.94 95.25)
 		)
 		(stroke
@@
 	(wire
 		(pts
-			(xy 148.59 92.71) (xy 148.59 93.98)
+			(xy 147.32 90.17) (xy 147.32 92.71)
 		)
 		(stroke
@@
 	(wire
 		(pts
-			(xy 139.7 90.17) (xy 138.43 90.17)
+			(xy 138.43 90.17) (xy 147.32 90.17)
 		)
 		(stroke
@@
 	(wire
 		(pts
-			(xy 283.21 86.36) (xy 284.48 86.36)
-		)
-		(stroke
-			(width 0)
-			(type default)
-		)
-	)
-	(wire
-		(pts
 			(xy 71.12 134.62) (xy 71.12 137.16)
 		)
@@
 	(rectangle
 		(start 129.54 186.69)
-		(end 204.47 231.14)
+		(end 208.28 231.14)
 		(stroke
 			(width 0)
@@
 		)
 	)
-	(text "Charge Pump -9V - ICL7660CBAZ"
+	(text "Charge Pump -9V - ICL7662CBAZ"
 		(exclude_from_sim no)
 		(at 288.544 61.468 0)
@@
 	)
 	(symbol
+		(lib_id "Measurement_Power_AC:ICL7662CBA-T")
+		(at 302.26 88.9 0)
+		(mirror y)
+		(unit 1)
+		(exclude_from_sim no)
+		(in_bom yes)
+		(on_board yes)
+		(dnp no)
+		(property "Reference" "U16"
+			(at 294.64 69.342 0)
+			(effects
+				(font
+					(size 1.27 1.27)
+				)
+			)
+		)
+		(property "Value" "ICL7662CBA-T"
+			(at 294.894 71.882 0)
+			(effects
+				(font
+					(size 1.27 1.27)
+				)
+			)
+		)
+		(property "Footprint" "Measure_Power_AC:SOIC-8"
+			(at 302.26 88.9 0)
+			(effects
+				(font
+					(size 1.27 1.27)
+				)
+				(justify bottom)
+				(hide yes)
+			)
+		)
+		(property "Datasheet" "https://www.analog.com/media/en/technical-documentation/data-sheets/icl7662-si7661.pdf"
+			(at 302.26 88.9 0)
+			(effects
+				(font
+					(size 1.27 1.27)
+				)
+				(hide yes)
+			)
+		)
+		(property "Description" "Điện áp vào: 4.5V ~ 20V, Điện áp ra: -Vin, 8-SOIC"
+			(at 302.26 88.9 0)
+			(effects
+				(font
+					(size 1.27 1.27)
+				)
+				(hide yes)
+			)
+		)
+		(property "Supply name" "ICL7662CBA"
+			(at 302.26 88.9 0)
+			(effects
+				(font
+					(size 1.27 1.27)
+				)
+				(hide yes)
+			)
+		)
+		(property "Supply part number" "ICL7662CBA"
+			(at 294.64 68.58 0)
+			(effects
+				(font
+					(size 1.27 1.27)
+				)
+				(hide yes)
+			)
+		)
+		(property "Supply URL" "https://www.thegioiic.com/icl7662cba"
+			(at 294.64 71.12 0)
+			(effects
+				(font
+					(size 1.27 1.27)
+				)
+				(hide yes)
+			)
+		)
+		(pin "3"
+		)
+		(pin "5"
+		)
+		(pin "1"
+		)
+		(pin "7"
+		)
+		(pin "8"
+		)
+		(pin "6"
+		)
+		(pin "4"
+		)
+		(pin "2"
+		)
+		(instances
+			(project ""
+				(path "/a4d4b55a-fae9-4c17-8d9b-0fae9d35e0cc/89f6d2d9-dbdb-44c3-92b1-b6c6afb905fd"
+					(reference "U16")
+					(unit 1)
+				)
+			)
+		)
+	)
+	(symbol
 		(lib_id "Measurement_Power_AC:Res_1K_0603_1%")
 		(at 372.11 76.2 0)
@@
 	(symbol
 		(lib_id "power:GND")
-		(at 148.59 93.98 0)
+		(at 147.32 92.71 0)
 		(unit 1)
 		(exclude_from_sim no)
@@
 		(fields_autoplaced yes)
 		(property "Reference" "#PWR0134"
-			(at 148.59 100.33 0)
+			(at 147.32 99.06 0)
 			(effects
 				(font
@@
 		)
 		(property "Value" "GND"
-			(at 148.59 99.06 0)
+			(at 147.32 97.79 0)
 			(effects
 				(font
@@
 		)
 		(property "Footprint" ""
-			(at 148.59 93.98 0)
+			(at 147.32 92.71 0)
 			(effects
 				(font
@@
 		)
 		(property "Datasheet" ""
-			(at 148.59 93.98 0)
+			(at 147.32 92.71 0)
 			(effects
 				(font
@@
 		)
 		(property "Description" "Power symbol creates a global label with name \"GND\" , ground"
-			(at 148.59 93.98 0)
+			(at 147.32 92.71 0)
 			(effects
 				(font
@@
 					(unit 1)
 				)
-			)
-		)
-	)
-	(symbol
-		(lib_id "Measurement_Power_AC:ICL7660CBAZ")
-		(at 302.26 88.9 0)
-		(mirror y)
-		(unit 1)
-		(exclude_from_sim no)
-		(in_bom yes)
-		(on_board yes)
-		(dnp no)
-		(property "Reference" "U16"
-			(at 294.64 68.58 0)
-			(effects
-				(font
-					(size 1.27 1.27)
-				)
-			)
-		)
-		(property "Value" "ICL7660CBAZ"
-			(at 294.64 71.12 0)
-			(effects
-				(font
-					(size 1.27 1.27)
-				)
-			)
-		)
-		(property "Footprint" "Measure_Power_AC:SOIC-8"
-			(at 321.31 110.744 0)
-			(effects
-				(font
-					(size 1.27 1.27)
-				)
-				(hide yes)
-			)
-		)
-		(property "Datasheet" "https://www.analog.com/media/en/technical-documentation/data-sheets/icl7662-si7661.pdf"
-			(at 301.752 110.49 0)
-			(effects
-				(font
-					(size 1.27 1.27)
-				)
-				(hide yes)
-			)
-		)
-		(property "Description" "Voltage Input: 1.5V ~ 10V, Voltage Output: -Vin, 8-SOIC"
-			(at 302.26 110.744 0)
-			(effects
-				(font
-					(size 1.27 1.27)
-				)
-				(hide yes)
-			)
-		)
-		(property "Supply name" "Thegioiic"
-			(at 300.99 110.49 0)
-			(effects
-				(font
-					(size 1.27 1.27)
-				)
-				(hide yes)
-			)
-		)
-		(property "Supply part number" "ICL7660CBAZ"
-			(at 300.99 110.49 0)
-			(effects
-				(font
-					(size 1.27 1.27)
-				)
-				(hide yes)
-			)
-		)
-		(property "Supply URL" "http://www.tme.vn/Product.aspx?id=848#page=pro_info"
-			(at 314.198 110.744 0)
-			(effects
-				(font
-					(size 1.27 1.27)
-				)
-				(hide yes)
-			)
-		)
-		(pin "3"
-		)
-		(pin "7"
-		)
-		(pin "5"
-		)
-		(pin "2"
-		)
-		(pin "1"
-		)
-		(pin "4"
-		)
-		(pin "6"
-		)
-		(pin "8"
-		)
-		(instances
-			(project ""
-				(path "/a4d4b55a-fae9-4c17-8d9b-0fae9d35e0cc/89f6d2d9-dbdb-44c3-92b1-b6c6afb905fd"
-					(reference "U16")
-					(unit 1)
-				)
